File: Shield TP Arduino/PRUEBA2.kicad_pcb (KiCad board)
At the start: 2 copper layers, 68.6 x 53.3 mm, 24 parts, among them J1 Power, J2 Digital/PWM, J3 Analog, J4 Digital/PWM, U2 LTC1050ACN8_PBF

Commit message: Update PRUEBA2.kicad_pcb
Parts:
- moved C4 12.3 mm to (162.0, 68.5), turned to 180 degrees
Routing:
- net CLK: track 42.7 -> 22.2 mm
Changed lines of the file:
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@@
 	(footprint "Capacitor_THT:C_Disc_D4.7mm_W2.5mm_P5.00mm"
 		(layer "F.Cu")
-		(at 150 66)
+		(at 162 68.5 180)
 		(descr "C, Disc series, Radial, pin pitch=5.00mm, diameter*width=4.7*2.5mm^2, Capacitor, http://www.vishay.com/docs/45233/krseries.pdf")
 		(tags "C Disc series Radial pin pitch 5.00mm diameter 4.7mm width 2.5mm Capacitor")
@@
 		(attr through_hole)
 		(fp_line
-			(start 0.03 -1.37)
-			(end 4.97 -1.37)
+			(start 4.97 1.37)
+			(end 0.03 1.37)
+			(stroke
+				(width 0.12)
+				(type solid)
+			)
+			(layer "F.SilkS")
+		)
+		(fp_line
+			(start 4.97 1.04)
+			(end 4.97 1.37)
+			(stroke
+				(width 0.12)
+				(type solid)
+			)
+			(layer "F.SilkS")
+		)
+		(fp_line
+			(start 4.97 -1.37)
+			(end 4.97 -1.04)
+			(stroke
+				(width 0.12)
+				(type solid)
+			)
+			(layer "F.SilkS")
+		)
+		(fp_line
+			(start 0.03 1.37)
+			(end 0.03 1.04)
 			(stroke
 				(width 0.12)
@@
 		)
 		(fp_line
-			(start 0.03 1.37)
-			(end 0.03 1.04)
-			(stroke
-				(width 0.12)
-				(type solid)
-			)
-			(layer "F.SilkS")
-		)
-		(fp_line
-			(start 4.97 -1.37)
-			(end 4.97 -1.04)
-			(stroke
-				(width 0.12)
-				(type solid)
-			)
-			(layer "F.SilkS")
-		)
-		(fp_line
-			(start 4.97 1.04)
-			(end 4.97 1.37)
-			(stroke
-				(width 0.12)
-				(type solid)
-			)
-			(layer "F.SilkS")
-		)
-		(fp_line
-			(start 4.97 1.37)
-			(end 0.03 1.37)
+			(start 0.03 -1.37)
+			(end 4.97 -1.37)
 			(stroke
 				(width 0.12)
@@
 		)
 		(pad "1" thru_hole circle
-			(at 0 0)
+			(at 0 0 180)
 			(size 1.6 1.6)
 			(drill 0.8)
@@
 		)
 		(pad "2" thru_hole circle
-			(at 5 0)
+			(at 5 0 180)
 			(size 1.6 1.6)
 			(drill 0.8)
@@
 	)
 	(segment
+		(start 163 67.5)
+		(end 163 55)
+		(width 0.8)
+		(layer "B.Cu")
+		(net 19)
+	)
+	(segment
 		(start 160.42 53.42)
 		(end 158.42 51.42)
@@
 	)
 	(segment
-		(start 150 58.5)
-		(end 150 66)
+		(start 161.42 53.42)
+		(end 160.75 53.42)
 		(width 0.8)
 		(layer "B.Cu")
@@
 	)
 	(segment
-		(start 158.42 49.2)
-		(end 158.42 48.42)
+		(start 162 68.5)
+		(end 163 67.5)
 		(width 0.8)
 		(layer "B.Cu")
@@
 	)
 	(segment
-		(start 143.5 47.918)
-		(end 143.5 52)
-		(width 0.8)
-		(layer "B.Cu")
-		(net 19)
-	)
-	(segment
-		(start 157.136 47.136)
-		(end 144.282 47.136)
-		(width 0.8)
-		(layer "B.Cu")
-		(net 19)
-	)
-	(segment
-		(start 144.282 47.136)
-		(end 143.5 47.918)
-		(width 0.8)
-		(layer "B.Cu")
-		(net 19)
-	)
-	(segment
-		(start 158.42 48.42)
-		(end 157.136 47.136)
-		(width 0.8)
-		(layer "B.Cu")
-		(net 19)
-	)
-	(segment
-		(start 143.5 52)
-		(end 150 58.5)
-		(width 0.8)
-		(layer "B.Cu")
+		(start 163 55)
+		(end 161.42 53.42)
+		(width 0.8)
+		(layer "B.Cu")
