File: Shield TP Arduino/PRUEBA2.kicad_pcb (KiCad board)
At the start: 2 copper layers, 68.6 x 53.3 mm, 24 parts, among them J1 Power, J2 Digital/PWM, J3 Analog, J4 Digital/PWM, U2 LTC1050ACN8_PBF

Commit message: Finish PCB files
Routing:
- net +5V: track 144.3 -> 179.2 mm
- net GND: track 9.22 -> 2.54 mm
- net SCK: track 39.0 -> 41.8 mm
- net TXD: track 46.6 -> 45.2 mm

Commit message: new update PCB
Routing:
- net SCL: track 19.1 -> 17.1 mm
